Commit message: finish test 2

File: irb120_robotiq85/irb120_robotiq85_gazebo/urdf/irb120_robotiq85_macro.xacro (robot description, xacro)
@@ -8,5 +8,5 @@
 	<xacro:include filename="$(find robotiq_85_description)/urdf/robotiq_85_gripper.urdf.xacro" />
 	<xacro:robotiq_85_gripper prefix="" parent="tool0">
-		<origin xyz="0 0 0" rpy="0 0 0" />
+		<origin xyz="0 0 0" rpy="0 -1.5707963267948966 0" />
 	</xacro:robotiq_85_gripper>
 </robot>
